Commit message: Adding in working model and moveit config packages for FANUC LRMate 200iD-7LC.

File: fanuc_lrmate200id_7lc_support/urdf/lrmate200id_7lc_macro.xacro (robot description, xacro)
@@ -110,5 +110,5 @@
     <link name="${prefix}tool0" />
     <joint name="${prefix}joint_1" type="revolute">
-      <origin xyz="0 0 0.330" rpy="0 0 0" />
+      <origin xyz="0 0 0.169" rpy="0 0 0" />
       <parent link="${prefix}base_link" />
       <child link="${prefix}link_1" />
@@ -117,40 +117,40 @@
     </joint>
     <joint name="${prefix}joint_2" type="revolute">
-      <origin xyz="0.050 0 0" rpy="0 0 0"/>
+      <origin xyz="0.05 0.001 0.1601" rpy="${-pi/2} 0 0"/>
       <parent link="${prefix}link_1" />
       <child link="${prefix}link_2" />
-      <axis xyz="0 1 0" />
+      <axis xyz="0 0 1" />
       <limit effort="0" lower="-1.745329" upper="2.530727" velocity="6.63" />
     </joint>
     <joint name="${prefix}joint_3" type="revolute">
-      <origin xyz="0 0 0.330" rpy="0 0 0"/>
+      <origin xyz="0 -0.44 0.001" rpy="0 0 ${-pi/2}"/>
       <parent link="${prefix}link_2" />
       <child link="${prefix}link_3" />
-      <axis xyz="0 -1 0" />
+      <axis xyz="0 0 -1" />
       <limit effort="0" lower="-2.450966" upper="4.886922" velocity="9.08" />
     </joint>
     <joint name="${prefix}joint_4" type="revolute">
-      <origin xyz="0 0 0.035" rpy="0 0 0"/>
+      <origin xyz="0.035055 0.0885 0.0034374" rpy="${-pi/2} 0 0"/>
       <parent link="${prefix}link_3"/>
       <child link="${prefix}link_4"/>
-      <axis xyz="-1 0 0"/>
+      <axis xyz="0 0 1"/>
       <limit effort="0" lower="-3.315" upper="3.315" velocity="9.60" />
     </joint>
     <joint name="${prefix}joint_5" type="revolute">
-      <origin xyz="0.335 0 0" rpy="0 0 0"/>
+      <origin xyz="0 0.00325000014011412 0.3299" rpy="${pi/2} 0 0"/>
       <parent link="${prefix}link_4"/>
       <child link="${prefix}link_5"/>
-      <axis xyz="0 -1 0"/>
+      <axis xyz="0 0 -1"/>
       <limit effort="0" lower="-2.18" upper="2.18" velocity="9.51" />
     </joint>
     <joint name="${prefix}joint_6" type="revolute">
-      <origin xyz="0.080 0 0" rpy="0 0 0"/>
+      <origin xyz="0 0.092 0" rpy="${-pi/2} 0 0"/>
       <parent link="${prefix}link_5"/>
       <child link="${prefix}link_6"/>
-      <axis xyz="-1 0 0"/>
+      <axis xyz="0 0 1"/>
       <limit effort="0" lower="-6.285" upper="6.285" velocity="17.45" />
     </joint>
     <joint name="${prefix}joint_6-tool0" type="fixed">
-      <origin xyz="0 0 0" rpy="${pi} ${-pi/2.0} 0" />
+      <origin xyz="0 0 0" rpy="0 0 ${pi}" />
       <parent link="${prefix}link_6" />
       <child link="${prefix}tool0" />
